Commit message: gazebo-ign

File: src/robot_description/urdf/waffle_base.xacro (robot description, xacro)
@@ -3,4 +3,7 @@
   <xacro:arg name="namespace" default=""/>
   <xacro:property name="namespace" value="$(arg namespace)"/>
+  <gazebo reference="${namespace}base_link">
+    <material>Gazebo/DarkGrey</material>
+  </gazebo>
   <link name="${namespace}base_footprint"/>
   <joint name="${namespace}base_joint" type="fixed">
@@ -36,4 +39,5 @@
     <origin xyz="0.0 0.144 0.023" rpy="-1.57 0 0"/>
     <axis xyz="0 0 1"/>
+    <dynamics damping="0.0" friction="0.0"/>
   </joint>
   <link name="${namespace}wheel_left_link">
@@ -64,4 +68,5 @@
     <origin xyz="0.0 -0.144 0.023" rpy="-1.57 0 0"/>
     <axis xyz="0 0 1"/>
+    <dynamics damping="0.0" friction="0.0"/>
   </joint>
   <link name="${namespace}wheel_right_link">
@@ -94,7 +99,7 @@
   <link name="${namespace}caster_back_right_link">
     <collision>
-      <origin xyz="0 0.001 0" rpy="0 0 0"/>
+      <origin xyz="0 0 0" rpy="0 0 0"/>
       <geometry>
-        <box size="0.030 0.009 0.020"/>
+        <sphere radius="0.015"/>
       </geometry>
     </collision>
@@ -112,7 +117,7 @@
   <link name="${namespace}caster_back_left_link">
     <collision>
-      <origin xyz="0 0.001 0" rpy="0 0 0"/>
+       <origin xyz="0 0 0" rpy="0 0 0"/>
       <geometry>
-        <box size="0.030 0.009 0.020"/>
+        <sphere radius="0.015"/>
       </geometry>
     </collision>

File: src/robot_description/urdf/waffle_diff_drive.xacro (robot description, xacro)
@@ -1,43 +1,46 @@
 <?xml version="1.0" ?>
 <robot xmlns:xacro="http://ros.org/wiki/xacro">
+  <!-- BACK RIGHT CASTER -->
   <gazebo reference="${namespace}caster_back_right_link">
-    <mu1>0.001</mu1>
-    <mu2>0.001</mu2>
-    <kp>1000000.0</kp>
-    <kd>100.0</kd>
+    <mu1>0.03</mu1>
+    <mu2>0.03</mu2>
+    <kp>150000.0</kp>
+    <kd>40.0</kd>
     <minDepth>0.001</minDepth>
-    <maxVel>1.0</maxVel>
+    <maxVel>0.5</maxVel>
     <material>Gazebo/FlatBlack</material>
   </gazebo>
+  <!-- BACK LEFT CASTER -->
   <gazebo reference="${namespace}caster_back_left_link">
-    <mu1>0.001</mu1>
-    <mu2>0.001</mu2>
-    <kp>1000000.0</kp>
-    <kd>100.0</kd>
+    <mu1>0.03</mu1>
+    <mu2>0.03</mu2>
+    <kp>150000.0</kp>
+    <kd>40.0</kd>
     <minDepth>0.001</minDepth>
-    <maxVel>1.0</maxVel>
+    <maxVel>0.5</maxVel>
     <material>Gazebo/FlatBlack</material>
   </gazebo>
+  <!-- LEFT WHEEL -->
   <gazebo reference="${namespace}wheel_left_link">
-    <mu1>10.0</mu1>
-    <mu2>10.0</mu2>
-    <kp>500000.0</kp>
-    <kd>10.0</kd>
+    <mu1>1.0</mu1>
+    <mu2>0.02</mu2>
+    <kp>200000.0</kp>
+    <kd>3.0</kd>
     <minDepth>0.001</minDepth>
-    <maxVel>0.1</maxVel>
+    <maxVel>0.05</maxVel>
     <fdir1>1 0 0</fdir1>
     <material>Gazebo/FlatBlack</material>
   </gazebo>
+  <!-- RIGHT WHEEL -->
   <gazebo reference="${namespace}wheel_right_link">
-    <mu1>10.0</mu1>
-    <mu2>10.0</mu2>
-    <kp>500000.0</kp>
-    <kd>10.0</kd>
+    <mu1>1.0</mu1>
+    <mu2>0.02</mu2>
+    <kp>200000.0</kp>
+    <kd>3.0</kd>
     <minDepth>0.001</minDepth>
-    <maxVel>0.1</maxVel>
+    <maxVel>0.05</maxVel>
     <fdir1>1 0 0</fdir1>
     <material>Gazebo/FlatBlack</material>
   </gazebo>
-  <!--
   <gazebo>
     <plugin name="turtlebot3_diff_drive" filename="libgazebo_ros_diff_drive.so">
@@ -58,4 +61,3 @@
     </plugin>
   </gazebo>
-  -->
 </robot>

File: src/robot_description/urdf/waffle_ros2_controller.xacro (robot description, xacro)
@@ -1,7 +1,9 @@
 <?xml version="1.0"?>
 <robot xmlns:xacro="http://www.ros.org/wiki/xacro">
-  <ros2_control name="GazeboSystem" type="system">
+  <xacro:arg name="namespace" default=""/>
+  <xacro:property name="namespace" value="$(arg namespace)"/>
+  <ros2_control name="IgnitionSystem" type="system">
     <hardware>
-      <plugin>gazebo_ros2_control/GazeboSystem</plugin>
+      <plugin>ign_ros2_control/IgnitionSystem</plugin>
     </hardware>
     <joint name="${namespace}wheel_left_joint">
@@ -23,5 +25,5 @@
   </ros2_control>
   <gazebo>
-    <plugin name="gazebo_ros2_control" filename="libgazebo_ros2_control.so">
+    <plugin filename="ign_ros2_control-system" name="ign_ros2_control::IgnitionROS2ControlPlugin">
       <parameters>$(find robot_description)/config/my_controllers.yaml</parameters>
     </plugin>

File: src/robot_description/urdf/waffle_sensors.xacro (robot description, xacro)
@@ -10,5 +10,9 @@
     <sensor name="tb3_imu" type="imu">
       <always_on>true</always_on>
-      <update_rate>200</update_rate>
+      <update_rate>50</update_rate>
+      <visualize>true</visualize>
+      <topic>imu</topic>
+      <frame_id>${namespace}imu_link</frame_id>
+      <ign_frame_id>${namespace}imu_link</ign_frame_id>
       <imu>
         <angular_velocity>
@@ -23,10 +27,4 @@
         </linear_acceleration>
       </imu>
-      <plugin name="turtlebot3_imu" filename="libgazebo_ros_imu_sensor.so">
-        <ros>
-          <namespace>${namespace}</namespace>
-          <remapping>~/out:=imu</remapping>
-        </ros>
-      </plugin>
     </sensor>
   </gazebo>
@@ -57,7 +55,11 @@
   </link>
   <gazebo reference="${namespace}base_scan">
-    <sensor name="hls_lfcd_lds" type="ray">
+    <sensor name="hls_lfcd_lds" type="gpu_lidar">
+      <topic>scan</topic>
       <always_on>true</always_on>
-      <visualize>true</visualize> <update_rate>5</update_rate>
+      <visualize>true</visualize>
+      <update_rate>5</update_rate>
+      <frame_id>${namespace}base_scan</frame_id>
+      <ign_frame_id>${namespace}base_scan</ign_frame_id>
       <ray>
         <scan>
@@ -80,12 +82,4 @@
         </noise>
       </ray>
-      <plugin name="turtlebot3_laserscan" filename="libgazebo_ros_ray_sensor.so">
-        <ros>
-          <namespace>${namespace}</namespace>
-          <remapping>~/out:=scan</remapping>
-        </ros>
-        <output_type>sensor_msgs/LaserScan</output_type>
-        <frame_name>base_scan</frame_name>
-      </plugin>
     </sensor>
   </gazebo>
@@ -135,7 +129,10 @@
   <gazebo reference="${namespace}camera_rgb_frame">
     <sensor name="camera" type="camera">
+      <topic>camera/image</topic>
       <always_on>true</always_on>
       <visualize>true</visualize>
       <update_rate>30</update_rate>
+      <frame_id>${namespace}camera_rgb_optical_frame</frame_id>
+      <ign_frame_id>${namespace}camera_rgb_optical_frame</ign_frame_id>
       <camera name="intel_realsense_r200">
         <horizontal_fov>1.02974</horizontal_fov>
@@ -155,12 +152,4 @@
         </noise>
       </camera>
-      <plugin name="camera_driver" filename="libgazebo_ros_camera.so">
-        <ros>
-          <namespace>${namespace}</namespace>
-        </ros>
-        <camera_name>camera</camera_name>
-        <frame_name>camera_rgb_optical_frame</frame_name>
-        <hack_baseline>0.07</hack_baseline>
-      </plugin>
     </sensor>
   </gazebo>
