Commit message: Rtab-map added

File: src/robot_description/urdf/waffle_sensors.xacro (robot description, xacro)
@@ -32,5 +32,5 @@
     <parent link="${namespace}base_link"/>
     <child link="${namespace}base_scan"/>
-    <origin xyz="-0.064 0 0.122" rpy="0 0 0"/>
+    <origin xyz="-0.064 0 0.30" rpy="0 0 0"/>
   </joint>
   <link name="${namespace}base_scan">
@@ -72,6 +72,6 @@
         </scan>
         <range>
-          <min>0.120</min>
-          <max>3.5</max>
+          <min>0.25</min>
+          <max>5</max>
           <resolution>0.015</resolution>
         </range>
@@ -138,6 +138,6 @@
         <horizontal_fov>1.02974</horizontal_fov>
         <image>
-          <width>1920</width>
-          <height>1080</height>
+          <width>640</width>
+          <height>480</height>
           <format>R8G8B8</format>
         </image>
